File: ram.kicad_sch (KiCad schematic)
At the start: 31 parts, among them SW3 SW_DIP_x08, SW4 SW_Push, U24 74LS245, U25 AS6C6264-55SIN, U26 74LS157, U27 74LS157, U28 74LS04, U29 74LS04, U30 74LS245, U31 74LS00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

Commit message: Add files via upload
RAM updated version with connected GND and Vcc.
Connections:
- net GND: now also U25.14 (VSS), U25.2 (A12), U25.21 (A10), U25.23 (A11), U25.24 (A9), U25.25 (A8), U25.3 (A7), U25.4 (A6), U25.5 (A5), U25.6 (A4)
- net VCC: now also U25.28 (VCC)
